Commit message: Updating the integration test.

File: moveit_experimental/jog_arm/test/arm_setup/urdf/test_six_dof_arm.xacro (robot description, xacro)
@@ -1,5 +1,5 @@
 <?xml version="1.0"?>
 <robot xmlns:xacro="http://www.ros.org/wiki/xacro" name="six_dof_arm" >
-    <xacro:include filename="$(find jog_arm)/test/arm_setup/urdf/test_six_dof_arm_macro.xacro"/>
+    <xacro:include filename="$(find moveit_experimental)/jog_arm/test/arm_setup/urdf/test_six_dof_arm_macro.xacro"/>
     <xacro:six_dof_arm prefix=""/>
 </robot>

File: moveit_experimental/jog_arm/test/arm_setup/urdf/test_six_dof_arm_macro.xacro (robot description, xacro)
@@ -6,5 +6,5 @@
             <visual>
                 <geometry>
-                    <mesh filename="package://jog_arm/test/arm_setup/meshes/robot_base_link.stl"/>
+                    <mesh filename="package://moveit_experimental/jog_arm/test/arm_setup/meshes/robot_base_link.stl"/>
                 </geometry>
                 <origin rpy="0.0 0 0.0" xyz="0 0 0"/>
@@ -17,5 +17,5 @@
             <visual>
                 <geometry>
-                    <mesh filename="package://jog_arm/test/arm_setup/meshes/robot_link_1.stl"/>
+                    <mesh filename="package://moveit_experimental/jog_arm/test/arm_setup/meshes/robot_link_1.stl"/>
                 </geometry>
                 <origin rpy="0.0 0 0.0" xyz="0 0 0"/>
@@ -28,5 +28,5 @@
             <visual>
                 <geometry>
-                    <mesh filename="package://jog_arm/test/arm_setup/meshes/robot_link_2.stl"/>
+                    <mesh filename="package://moveit_experimental/jog_arm/test/arm_setup/meshes/robot_link_2.stl"/>
                 </geometry>
                 <origin rpy="0.0 0 0.0" xyz="0 0 0"/>
@@ -39,5 +39,5 @@
             <visual>
                 <geometry>
-                    <mesh filename="package://jog_arm/test/arm_setup/meshes/robot_link_3.stl"/>
+                    <mesh filename="package://moveit_experimental/jog_arm/test/arm_setup/meshes/robot_link_3.stl"/>
                 </geometry>
                 <origin rpy="0.0 0 0.0" xyz="0 0 0"/>
@@ -50,5 +50,5 @@
             <visual>
                 <geometry>
-                    <mesh filename="package://jog_arm/test/arm_setup/meshes/robot_link_4.stl"/>
+                    <mesh filename="package://moveit_experimental/jog_arm/test/arm_setup/meshes/robot_link_4.stl"/>
                 </geometry>
                 <origin rpy="0.0 0 0.0" xyz="0 0 0"/>
@@ -61,5 +61,5 @@
             <visual>
                 <geometry>
-                    <mesh filename="package://jog_arm/test/arm_setup/meshes/robot_link_5.stl"/>
+                    <mesh filename="package://moveit_experimental/jog_arm/test/arm_setup/meshes/robot_link_5.stl"/>
                 </geometry>
                 <origin rpy="0.0 0 0.0" xyz="0 0 0"/>
@@ -72,5 +72,5 @@
             <visual>
                 <geometry>
-                    <mesh filename="package://jog_arm/test/arm_setup/meshes/robot_link_6.stl"/>
+                    <mesh filename="package://moveit_experimental/jog_arm/test/arm_setup/meshes/robot_link_6.stl"/>
                 </geometry>
                 <origin rpy="0.0 0 0.0" xyz="0 0 0"/>
